File: pcb/smoke_extractorV1_1/smoke_extractorV1_1.kicad_sch (KiCad schematic)
At the start: 48 parts, among them J1 USB_C_Receptacle, J2 Screw_Terminal_01x02, Q1 AO3400A, U1 LMV331, U2 RA11131100, U3 MP1542, U4 LMV331, U5 LMV331, U6 STBP120

Commit message: Removed the voltage IC and one mounting hole. Missing boost converter conns only.
Parts:
- removed C8, C9: 10u, Capacitor_SMD:C_0805_2012Metric_Pad1.18x1.45mm_HandSolder, symbol Device:C
- removed H4: MountingHole_Pad, MountingHole:MountingHole_3.2mm_M3_ISO7380_Pad, symbol Mechanical:MountingHole_Pad
- removed R20: 100k, Resistor_SMD:R_0603_1608Metric_Pad0.98x0.95mm_HandSolder, symbol Device:R
- removed U6: STBP120, Package_DFN_QFN:TDFN-10-1EP_2x3mm_P0.5mm_EP0.9x2mm_ThermalVias, symbol CustomSymbols:STBP120
- D4: footprint LED_SMD:LED_0201_0603Metric_Pad0.64x0.40mm_HandSolder -> LED_SMD:LED_0603_1608Metric_Pad1.05x0.95mm_HandSolder
Connections:
- net VBUS: now also J1.A4 (VBUS), J1.A9 (VBUS), J1.B4 (VBUS), J1.B9 (VBUS)
- no-connect marks 11 -> 10

Commit message: Schematic as pdf
Parts:
- R5: value 4.7k -> 47k
Changed lines of the file:
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@@
       (effects (font (size 1.27 1.27)) (justify right))
     )
-    (property "Value" "4.7k" (id 1) (at 100.33 35.56 0)
+    (property "Value" "47k" (id 1) (at 100.33 35.56 0)
       (effects (font (size 1.27 1.27)) (justify right))
     )
@@
     )
     (path "/928b81d5-4f5c-43d6-adf5-dda019181b73"
-      (reference "R5") (unit 1) (value "4.7k") (footprint "Resistor_SMD:R_0603_1608Metric_Pad0.98x0.95mm_HandSolder")
+      (reference "R5") (unit 1) (value "47k") (footprint "Resistor_SMD:R_0603_1608Metric_Pad0.98x0.95mm_HandSolder")
     )
     (path "/b683cc23-b225-4f7c-ab01-f58eb518a6d4"

Commit message: Version 1.2
Parts:
- added D6: SS34, Diode_SMD:Nexperia_CFP3_SOD-123W, symbol Device:D
- R10: value 4k7 -> 5k1
- R12: value 86.6k -> 1k
- R17: value 10k -> 12k
- R18, R19, R6: value 4.7k -> 5k1
- R9: value 330 -> 100
- U1, U4, U5: footprint Package_TO_SOT_SMD:SOT-353_SC-70-5_Handsoldering -> Package_TO_SOT_SMD:SOT-23-5_HandSoldering
Connections:
- net GND: now also Q1.2 (S); no longer C2.2, C3.2, C5.2, D4.1 (K), J2.2 (Pin_2), R14.2, R15.2, R17.2, U3.4 (GND)
- net VBUS: now also U2.1 (IN), D6.1 (K); no longer Q1.3 (D)
- removed net VBUS_OPEN: Q1.2 (S), U2.1 (IN)
- new net VBUS_DRAIN: C2.2, C3.2, C5.2, D4.1 (K), D6.2 (A), J2.2 (Pin_2), Q1.3 (D), R14.2, R15.2, R17.2, U3.4 (GND)
Other:
- moved on the sheet: D1, D2, D3, Q1, R10, R9
