File: pcb/1v1/smoke_extractorV1_1.kicad_sch (KiCad schematic)
At the start: 44 parts, among them J1 USB_C_Receptacle, J2 Screw_Terminal_01x02, Q1 AO3400A, U1 LMV331, U2 RA11131100, U3 MP1542, U4 LMV331, U5 LMV331

Commit message: smoke extractor 2.0
Parts:
- removed D1, D2, D3: D, Diode_SMD:D_SOD-523, symbol Device:D
- removed D5, D6: SS34, Diode_SMD:Nexperia_CFP3_SOD-123W, symbol Device:D
- removed H3: MountingHole_Pad, MountingHole:MountingHole_3.2mm_M3_ISO7380_Pad, symbol Mechanical:MountingHole_Pad
- removed J1: USB_C_Receptacle, CustomFootprints:USB4120-03-C, symbol Connector:USB_C_Receptacle
- removed Q1: AO3400A, Package_TO_SOT_SMD:SOT-23, symbol Transistor_FET:AO3400A
- removed U1, U4, U5: LMV331, Package_TO_SOT_SMD:SOT-23-5_HandSoldering, symbol Comparator:LMV331
- removed U3: MP1542, Package_SO:MSOP-8_3x3mm_P0.65mm, symbol CustomSymbols:MP1542
- added C8: 22u, Capacitor_SMD:C_0805_2012Metric_Pad1.18x1.45mm_HandSolder, symbol Device:C
- added D1: LED, LED_SMD:LED_0603_1608Metric_Pad1.05x0.95mm_HandSolder, symbol Device:LED
- added D10, D6, D9: SS14, Diode_SMD:D_SMA_Handsoldering, symbol Device:D_Schottky
- added D2, D3, D5: 3mmWhite, LED_THT:LED_D3.0mm, symbol Device:LED
- added D7: RLED, LED_SMD:LED_0603_1608Metric_Pad1.05x0.95mm_HandSolder, symbol Device:LED
- added D8: GLED, LED_SMD:LED_0603_1608Metric_Pad1.05x0.95mm_HandSolder, symbol Device:LED
- added IC1: DW01A, Package_TO_SOT_SMD:SOT-23-6_Handsoldering, symbol DW01A:DW01A
- added Q1: FDN336P, Package_TO_SOT_SMD:SOT-23, symbol Transistor_FET:FDN340P
- added R20: 100, Resistor_SMD:R_0805_2012Metric_Pad1.20x1.40mm_HandSolder, symbol Device:R
- added R21: 44.2k, Resistor_SMD:R_0603_1608Metric_Pad0.98x0.95mm_HandSolder, symbol Device:R
- added R22: 5k1, Resistor_SMD:R_0603_1608Metric_Pad0.98x0.95mm_HandSolder, symbol Device:R
- added R23: 1k, Resistor_SMD:R_0603_1608Metric_Pad0.98x0.95mm_HandSolder, symbol Device:R
- added SW1: SW_Push, Button_Switch_SMD:SW_SPST_SKQG_WithStem, symbol Switch:SW_Push
- added TP1, TP2: TestPoint, TestPoint:TestPoint_Pad_2.0x2.0mm, symbol Connector:TestPoint
- added U1: USB-TYPE-C-31-M-15, CustomFootprints:USB-TYPE-C-31-M-15, symbol CustomSymbols:USB-TYPE-C-31-M-15
- added U3: LM324DT, Package_SO:SOIC127P600X175-14N, symbol LM324DT:LM324DT
- added U4: TPS613222ADBV, Package_TO_SOT_SMD:SOT-23-5, symbol Regulator_Switching:TPS613222ADBV
- added U5: TP4056, Package_SO:SOP-8_3.9x4.9mm_P1.27mm, symbol TP4046:TP4056
- added U6: 18350-HOLDER, CustomFootprints:18350-Holder, symbol CustomSymbols:18350-HOLDER
- added U7: ME2149FM5G, Package_TO_SOT_SMD:SOT-23-5_HandSoldering, symbol CustomSymbols:ME2149FM5G
- added U8: FH8205, Package_TO_SOT_SMD:SOT-23-6_Handsoldering, symbol Transistor_FET:FH8205
- C1, C7: LCSC (none) -> C30926
- C2: value 10u -> 120p; footprint Capacitor_SMD:C_0805_2012Metric_Pad1.18x1.45mm_HandSolder -> Capacitor_SMD:C_0603_1608Metric_Pad1.08x0.95mm_HandSolder; LCSC (none) -> C1643
- C3: value 10n -> 10u; LCSC (none) -> C19702
- C4: value 2.2n -> 10u; LCSC (none) -> C19702
- C5: footprint Capacitor_SMD:C_0805_2012Metric_Pad1.18x1.45mm_HandSolder -> Capacitor_SMD:C_0603_1608Metric_Pad1.08x0.95mm_HandSolder; LCSC (none) -> C19702
- C6: value 0.1u -> 10u; LCSC (none) -> C19702
- D4: value LED -> 3mmWhite; footprint LED_SMD:LED_0603_1608Metric_Pad1.05x0.95mm_HandSolder -> LED_THT:LED_D3.0mm; LCSC (none) -> C86881
- L1: value 4.7u -> 3.3u; footprint Inductor_SMD:L_1008_2520Metric_Pad1.43x2.20mm_HandSolder -> Inductor_SMD:L_Wuerth_WE-PD2-Typ-MS; LCSC (none) -> C2929417
- R1, R7: value 47k -> 3k6; LCSC (none) -> C103578
- R10: LCSC (none) -> C178023
- R11, R13: value 5.1k -> 1k; LCSC (none) -> C328340
- R12: LCSC (none) -> C328340
- R14: value 100k -> 1k; LCSC (none) -> C328340
- R15: value 15k -> 1k; LCSC (none) -> C328340
- R16: value 86.6k -> 1.2k; LCSC (none) -> C118396
- R17: value 12k -> 5; footprint Resistor_SMD:R_0603_1608Metric_Pad0.98x0.95mm_HandSolder -> Resistor_SMD:R_0805_2012Metric_Pad1.20x1.40mm_HandSolder; LCSC (none) -> C17724; descp (none) -> 5 OHM 5% 1/3W 0805
- R18, R19: value 5k1 -> 1k; LCSC (none) -> C328340
- R2: value 6k8 -> 16k; LCSC (none) -> C4210
- R3, R5: value 47k -> 1k8; LCSC (none) -> C25958
- R4: value 4k7 -> 5k1; LCSC (none) -> C178023
- R6: value 5k1 -> 3k6; LCSC (none) -> C103578
- R8: value 7k6 -> 5k1; LCSC (none) -> C178023
- R9: value 100 -> 5k1; LCSC (none) -> C178023
- U2: value RA11131100 -> SDDJE; footprint CustomFootprints:RA11131100 -> CustomFootprints:SDDJE; LCSC (none) -> C358626
Connections:
- net CC2 is gone; now on an unnamed net: R13.2
- net D- is gone; now on net +5V: R5.1
- net GND: now also C3.2, C4.2, C5.2, J2.2 (Pin_2), R16.2, R2.2, R4.2, R6.2, R8.2, R9.2, C8.2, D1.1 (K), R22.2, R23.1, SW1.1, U1.1 (GND), U3.11 (VCC-), U4.2 (GND), U5.1 (TEMP), U5.3 (GND), U7.3 (GND), U8.3 (S2); no longer C7.2, R11.1, R13.1, R2.1, R4.1, R5.2, R8.1
- net VBUS: now also R11.1, D7.2 (A), D8.2 (A), D9.2 (A), Q1.1 (G), U1.2 (VCC), U5.4 (VCC), U5.8 (CE); no longer C6.1, C7.1, R1.2, R18.2, R19.2, R3.2, R6.2, R7.2, U2.1 (IN)
- net +5V: now reaches C4.1
- net +5V: now also C2.2, C3.1, C5.1, R1.1, R3.1, R7.1, U2.1 (IN), D6.1 (K), U3.4 (VCC+), U4.4 (VOUT)
- net VSPLY: now reaches R17.1
- net VSPLY: now also D6.2 (A), D9.1 (K), Q1.2 (S), TP2.1, U4.1 (SW); no longer R16.2
- net at L1.2: now also D10.2 (A), U7.2 (LX)
- net at R15.1: now also U3.14 (OUT4); no longer C4.2
- net at R10.1: now also U1.3 (CC1); no longer R9.1
- net at D4.2 (A): no longer R12.2
- net CC1: no longer names the net of R11.2
- net CC1: now also D1.2 (A)
- net CC1_DET: no longer names the net of R18.1
- net CC1_DET: now also D7.1 (K)
- net CC2_DET: no longer names the net of R19.1
- net CC2_DET: now also D8.1 (K)
- net CHG_DET: no longer names the net of R6.1
- net CHG_DET: now also R5.2, U3.9 (NEG3)
- removed net D+: R1.1, R2.2
- removed net VBOOST_OUT: C5.1, J2.1 (Pin_1), R16.1
- removed net VBUS_DRAIN: C2.2, C3.2, C5.2, D4.1 (K), J2.2 (Pin_2), R14.2, R15.2, R17.2
- removed net VBUS_SWITCH: C2.1, L1.1, R12.1, R14.1, U2.2 (OUT)
- removed net VDAT_REF: R3.1, R4.2
- removed net V_CC_REF: R7.1, R8.2
- new net: R3.2, R4.1, U3.6 (NEG_2)
- new net: R13.1, U3.7 (OUT2)
- new net: R16.1, U5.2 (PROG)
- new net: D2.1 (K), D3.1 (K), D4.1 (K), D5.1 (K), SW1.2
- new net: D5.2 (A), R12.2
- new net: R19.2, U5.6 (~{STDBY})
- new net: C7.2, IC1.6 (GND), U6.2 (V-), U8.1 (S1)
- new net: IC1.1 (OD), U8.4 (G1)
- new net: IC1.3 (OC), U8.6 (G2)
- new net: C2.1, R17.2
- new net: R21.2, R22.1, U7.5 (FB)
- new net: D3.2 (A), R14.2
- new net: R1.2, R2.1, U3.2 (NEG_1)
- new net: R18.2, U5.7 (~{CHRG})
- new net: C7.1, IC1.5 (VCC), R20.2
- new net: R12.1, U3.1 (OUT1)
- new net: R7.2, R8.1, U3.13 (NEG_4)
- new net: R14.1, U3.8 (OUT3)
- new net: IC1.2 (CS), R23.2
- new net: R9.1, U1.4 (CC2)
- new net: D2.2 (A), R15.2
- new net +12V: C8.1, D10.1 (K), J2.1 (Pin_1), R21.1
- new net V5_SWITCH: C6.1, L1.1, TP1.1, U2.2 (OUT), U7.1 (CE), U7.4 (VDD)
- new net VBAT+PROTECT: Q1.3 (D), R20.1, U3.10 (POS_3), U3.12 (POS_4), U3.3 (POS_1), U3.5 (POS_2), U5.5 (BAT), U6.1 (V+)
- no-connect marks 10 -> 6
Other:
- note added: "2.9V"
- note added: "3.3V"
- note added: "3.7V"
- note added: "4.1V"
- note added: "About the TP4056: https://www.best-microcontroller-projects.com/tp4056.html"
- note added: "Based on 5V"
- note added: "ME2149: https://datasheet.lcsc.com/lcsc/1808091834_MICRONE-Nanjing-Micro-One-Elec-ME2149FM5G_C236786.pdf From: https://lygte-info.dk/review/Power%205V%20to%2012V%206W%20boost%20converter%20UK.html"
- note added: "OK"
- note added: "R1 = R2(Vout - Vb) / Vb R1+R2<50K Vout = 12, Vb = 1.25 R1 = 8.6 * R2"
- note added: "R2"
- note added: "Sch Diode 1A >"
- note added: "To calculate the R1/R2 pair: https://damien.douxchamps.net/elec/resdiv/"
- note added: "USB"
- note added: "USB-C Receptacle: https://jlcpcb.com/partdetail/Korean_HropartsElec-TYPE_C_31_M15/C223908"
- note removed: "BOOST"
- note removed: "Boost Converter: https://www.digikey.se/en/products/detail/monolithic-power-systems-inc/MP1542DK-LF-Z/5291722"
- note removed: "CC LINES COMPARATOR"
- note removed: "Comparator: https://www.diodes.com/assets/Datasheets/LMV331_393.pdf"
- note removed: "DATA LINES COMPARATOR"
- note removed: "Double check the Vref!"
- note removed: "OVERVOLTAGE PROTECTION"
- note removed: "Outputs 0.4V"
- note removed: "Outputs 0.6V"
- note removed: "Outputs 0.7V"
- note removed: "USB-C Receptacle: https://www.digikey.se/en/products/detail/gct/USB4120-03-C/13547390"
- note removed: "V- > V+ then Vout = 0V V- < V+ then Vout = 5V V- = Vref V+ = Vin"
- note removed: "VBUS LOGIC"
- note removed: "VDAT_REF should have 0.4V at the terminals"
- note removed: "VDP_SRC should output 0.6V to D+"
- moved on the sheet: H2

Commit message: version 2.01 ready to order
Parts:
- added L2: 2.2u, Inductor_SMD:L_Coilcraft_LPS4018, symbol Device:L
- D10, D6, D9: footprint Diode_SMD:D_SMA_Handsoldering -> Diode_SMD:D_SMA
Connections:
- net VBAT+PROTECT: now also Q1.2 (S); no longer Q1.3 (D)
- net VSPLY: now also Q1.3 (D), L2.1; no longer D6.2 (A), Q1.2 (S), R17.1, U4.1 (SW)
- new net: D6.2 (A), L2.2, R17.1, U4.1 (SW)
Other:
- moved on the sheet: Q1
Changed lines of the file:
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@@
   (title_block
     (title "Smoke Extractor Schematic")
-    (date "2022-09-10")
-    (rev "2.0")
+    (date "2023-05-06")
+    (rev "2.01")
     (company "Nuno Nogueira")
     (comment 1 "1.2 - Changed LMV331 footprint, resistors values (from 4k7 to 5k1), changed VBUS circuit")
     (comment 2 "2.0 - Completely changed internals. Added battery LED feedback, battery charging IC, battery protection, step-up 5V, step-up 12V")
+    (comment 3 "2.01 - Fixed P-ch mosfet Drain/Source side and added inductor before the 5V boost converter")
   )
   (junction (at 212.09 125.73) (diameter 0) (color 0 0 0 0)
@@
     (stroke (width 0) (type default) (color 0 0 0 0))
   )
+  (wire (pts (xy 123.444 25.4) (xy 123.444 33.02))
+    (stroke (width 0) (type default) (color 0 0 0 0))
+  )
   (wire (pts (xy 85.09 30.48) (xy 86.36 30.48))
     (stroke (width 0) (type default) (color 0 0 0 0))
@@
   )
   (wire (pts (xy 137.16 19.05) (xy 137.16 25.4))
+    (stroke (width 0) (type default) (color 0 0 0 0))
+  )
+  (wire (pts (xy 123.444 33.02) (xy 124.46 33.02))
     (stroke (width 0) (type default) (color 0 0 0 0))
   )
@@
     )
   )
-  (global_label "VSPLY" (shape input) (at 132.08 33.02 180) (fields_autoplaced)
-    (effects (font (size 1.27 1.27)) (justify right))
-    (property "Intersheet References" "${INTERSHEET_REFS}" (id 0) (at 123.9821 32.9406 0)
-      (effects (font (size 1.27 1.27)) (justify right) hide)
+  (global_label "VSPLY" (shape input) (at 123.444 25.4 90) (fields_autoplaced)
+    (effects (font (size 1.27 1.27)) (justify left))
+    (property "Intersheet References" "${INTERSHEET_REFS}" (id 0) (at 123.5234 17.3021 90)
+      (effects (font (size 1.27 1.27)) (justify left) hide)
     )
   )
@@
       (effects (font (size 1.27 1.27)) (justify right))
     )
-    (property "Footprint" "Diode_SMD:D_SMA_Handsoldering" (id 2) (at 204.47 60.96 0)
+    (property "Footprint" "Diode_SMD:D_SMA" (id 2) (at 204.47 60.96 0)
       (effects (font (size 1.27 1.27)) hide)
     )
@@
     (pin "6")
   )
+  (symbol (lib_id "Device:L") (at 128.27 33.02 90) (unit 1)
+    (in_bom yes) (on_board yes) (fields_autoplaced)
+    (property "Reference" "L2" (id 0) (at 128.27 28.8122 90))
+    (property "Value" "2.2u" (id 1) (at 128.27 31.3491 90))
+    (property "Footprint" "Inductor_SMD:L_Coilcraft_LPS4018" (id 2) (at 128.27 33.02 0)
+      (effects (font (size 1.27 1.27)) hide)
+    )
+    (property "Datasheet" "https://datasheet.lcsc.com/lcsc/2201121400_SHOU-HAN-CY43-2-2UH_C2929416.pdf" (id 3) (at 128.27 33.02 0)
+      (effects (font (size 1.27 1.27)) hide)
+    )
+    (property "LCSC" "C2929416" (id 4) (at 128.27 33.02 90)
+      (effects (font (size 1.27 1.27)) hide)
+    )
+    (pin "1")
+    (pin "2")
+  )
   (symbol (lib_id "Device:C") (at 153.67 19.05 90) (unit 1)
     (in_bom yes) (on_board yes) (fields_autoplaced)
@@
     (property "Reference" "D6" (id 0) (at 148.9075 20.4302 0))
     (property "Value" "SS14" (id 1) (at 148.9075 22.9671 0))
-    (property "Footprint" "Diode_SMD:D_SMA_Handsoldering" (id 2) (at 148.59 25.4 0)
+    (property "Footprint" "Diode_SMD:D_SMA" (id 2) (at 148.59 25.4 0)
       (effects (font (size 1.27 1.27)) hide)
     )
@@
     (property "Reference" "D10" (id 0) (at 231.4575 120.7602 0))
     (property "Value" "SS14" (id 1) (at 231.4575 123.2971 0))
-    (property "Footprint" "Diode_SMD:D_SMA_Handsoldering" (id 2) (at 231.14 125.73 0)
+    (property "Footprint" "Diode_SMD:D_SMA" (id 2) (at 231.14 125.73 0)
       (effects (font (size 1.27 1.27)) hide)
     )
@@
     (pin "2")
   )
-  (symbol (lib_id "Transistor_FET:FDN340P") (at 196.85 63.5 90) (mirror x) (unit 1)
+  (symbol (lib_id "Transistor_FET:FDN340P") (at 196.85 63.5 270) (unit 1)
     (in_bom yes) (on_board yes) (fields_autoplaced)
     (property "Reference" "Q1" (id 0) (at 196.85 69.9754 90))
     (property "Value" "FDN336P" (id 1) (at 196.85 72.5123 90))
-    (property "Footprint" "Package_TO_SOT_SMD:SOT-23" (id 2) (at 198.755 68.58 0)
+    (property "Footprint" "Package_TO_SOT_SMD:SOT-23" (id 2) (at 194.945 68.58 0)
       (effects (font (size 1.27 1.27) italic) (justify left) hide)
     )
@@
     )
     (path "/5841b95e-a681-462d-b330-355b23ba28f1"
-      (reference "D6") (unit 1) (value "SS14") (footprint "Diode_SMD:D_SMA_Handsoldering")
+      (reference "D6") (unit 1) (value "SS14") (footprint "Diode_SMD:D_SMA")
     )
     (path "/48aa545d-0def-452f-bcec-b9f3b4549c0c"
@@
     )
     (path "/01ee1696-6f00-4208-8095-ed95fe08d7ea"
-      (reference "D9") (unit 1) (value "SS14") (footprint "Diode_SMD:D_SMA_Handsoldering")
+      (reference "D9") (unit 1) (value "SS14") (footprint "Diode_SMD:D_SMA")
     )
     (path "/6b3ae554-8492-438e-8e4a-ad5153dbc108"
-      (reference "D10") (unit 1) (value "SS14") (footprint "Diode_SMD:D_SMA_Handsoldering")
+      (reference "D10") (unit 1) (value "SS14") (footprint "Diode_SMD:D_SMA")
     )
     (path "/c05ca9f6-0404-4595-a216-dc8bde49db98"
@@
       (reference "L1") (unit 1) (value "3.3u") (footprint "Inductor_SMD:L_Wuerth_WE-PD2-Typ-MS")
     )
+    (path "/4d2c82eb-9afb-4f24-95d3-a5cb04b3d4e3"
+      (reference "L2") (unit 1) (value "2.2u") (footprint "Inductor_SMD:L_Coilcraft_LPS4018")
+    )
     (path "/f4fa2feb-5dd0-4a82-8393-5df29c40d818"

Commit message: v2.02
Parts:
- removed J2: Screw_Terminal_01x02, TerminalBlock:TerminalBlock_bornier-2_P5.08mm, symbol Connector:Screw_Terminal_01x02
- removed R6, R7: 3k6, Resistor_SMD:R_0603_1608Metric_Pad0.98x0.95mm_HandSolder, symbol Device:R
- removed R8: 5k1, Resistor_SMD:R_0603_1608Metric_Pad0.98x0.95mm_HandSolder, symbol Device:R
- added J13: JST XH, Connector_JST:JST_PH_S2B-PH-K_1x02_P2.00mm_Horizontal, symbol Connector:Conn_01x02_Socket
- R2: value 16k -> 1k; LCSC C4210 -> C328340
- R23: value 1k -> 3k3
- R3: value 1k8 -> 1k; LCSC C25958 -> C328340
- R4: value 5k1 -> 1k; LCSC C178023 -> C328340
- R5: value 1k8 -> 10k; LCSC C25958 -> C2930027
Connections:
- net +12V: now also J13.1 (Pin_1)
- net +5V: no longer R3.1, R5.1
- net GND: now also R5.2, J13.2 (Pin_2); no longer R2.2, R4.2
- net at R3.2, R4.1: now also U3.9 (NEG3); no longer U3.6 (NEG_2)
- net at U3.13 (NEG_4): now also R4.2, R5.1
- new net: R2.2, R3.1, U3.6 (NEG_2)
Other:
- note added: "3.9V"
- note added: "3V"
- note removed: "2.9V"
- note removed: "3.3V"
- note removed: "3.7V"
- note removed: "4.1V"

Commit message: version 2,03 and 2.04!
Parts:
- removed J13: JST XH, Connector_JST:JST_PH_S2B-PH-K_1x02_P2.00mm_Horizontal, symbol Connector:Conn_01x02_Socket
- removed R23: 3k3, Resistor_SMD:R_0603_1608Metric_Pad0.98x0.95mm_HandSolder, symbol Device:R
- added J1, J2: Conn_01x01_Socket, TestPoint:TestPoint_Pad_2.5x2.5mm, symbol Connector:Conn_01x01_Socket
- added R6: 1k, Resistor_SMD:R_0603_1608Metric_Pad0.98x0.95mm_HandSolder, symbol Device:R
Connections:
- net +12V: now also J1.1 (Pin_1)
- net GND: now also J2.1 (Pin_1), R6.1
- net at IC1.2 (CS): now also R6.2
Changed lines of the file:
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@@
   (title_block
     (title "Smoke Extractor Schematic")
-    (date "2023-09-24")
-    (rev "2.02")
+    (date "2023-11-30")
+    (rev "2.04")
     (company "Nuno Nogueira")
     (comment 1 "1.2 - Changed LMV331 footprint, resistors values (from 4k7 to 5k1), changed VBUS circuit")
@@
     (comment 3 "2.01 - Fixed P-ch mosfet Drain/Source side and added inductor before the 5V boost converter")
     (comment 4 "2.02 - Decreased the number of resitors on the LM324")
+    (comment 5 "2.03 - Simplified comparator circuit")
+    (comment 6 "2.04 - R6 from 3k3 to 1k.")
   )
   (junction (at 212.09 125.73) (diameter 0) (color 0 0 0 0)
@@
     )
   )
+  (symbol (lib_id "Device:R") (at 262.89 83.82 270) (unit 1)
+    (in_bom yes) (on_board yes) (dnp no) (fields_autoplaced)
+    (property "Reference" "R6" (at 262.89 78.6597 90)
+      (effects (font (size 1.27 1.27)))
+    )
+    (property "Value" "1k" (at 262.89 81.0839 90)
+      (effects (font (size 1.27 1.27)))
+    )
+    (property "Footprint" "Resistor_SMD:R_0603_1608Metric_Pad0.98x0.95mm_HandSolder" (at 262.89 82.042 90)
+      (effects (font (size 1.27 1.27)) hide)
+    )
+    (property "Datasheet" "https://datasheet.lcsc.com/lcsc/1811151159_Resistor-Today-AECR0603F1K00K9_C328340.pdf" (at 262.89 83.82 0)
+      (effects (font (size 1.27 1.27)) hide)
+    )
+    (property "LCSC" "C328340" (at 262.89 83.82 90)
+      (effects (font (size 1.27 1.27)) hide)
+    )
+    (pin "1")
+    (pin "2")
+    (instances
+      (project "smoke_extractorV1_1"
+        (path "/9c1091b5-dc9c-4275-a62f-af3d6f92e0db"
+          (reference "R6") (unit 1)
+        )
+      )
+    )
+  )
   (symbol (lib_id "Mechanical:MountingHole_Pad") (at 152.4 167.64 0) (unit 1)
     (in_bom yes) (on_board yes) (dnp no) (fields_autoplaced)
@@
     )
   )
+  (symbol (lib_id "Connector:Conn_01x01_Socket") (at 129.54 128.27 90) (unit 1)
+    (in_bom yes) (on_board yes) (dnp no)
+    (property "Reference" "J2" (at 128.27 126.365 90)
+      (effects (font (size 1.27 1.27)) (justify right))
+    )
+    (property "Value" "Conn_01x01_Socket" (at 135.255 127.635 0)
+      (effects (font (size 1.27 1.27)) (justify right))
+    )
+    (property "Footprint" "TestPoint:TestPoint_Pad_2.5x2.5mm" (at 129.54 128.27 0)
+      (effects (font (size 1.27 1.27)) hide)
+    )
+    (property "Datasheet" "~" (at 129.54 128.27 0)
+      (effects (font (size 1.27 1.27)) hide)
+    )
+    (pin "1")
+    (instances
+      (project "smoke_extractorV1_1"
+        (path "/9c1091b5-dc9c-4275-a62f-af3d6f92e0db"
+          (reference "J2") (unit 1)
+        )
+      )
+    )
+  )
   (symbol (lib_id "CustomSymbols:USB-TYPE-C-31-M-15") (at 34.29 102.87 0) (unit 1)
     (in_bom yes) (on_board yes) (dnp no) (fields_autoplaced)
@@
     )
   )
-  (symbol (lib_id "Device:R") (at 262.89 83.82 270) (unit 1)
-    (in_bom yes) (on_board yes) (dnp no) (fields_autoplaced)
-    (property "Reference" "R23" (at 262.89 79.1042 90)
-      (effects (font (size 1.27 1.27)))
-    )
-    (property "Value" "3k3" (at 262.89 81.6411 90)
-      (effects (font (size 1.27 1.27)))
-    )
-    (property "Footprint" "Resistor_SMD:R_0603_1608Metric_Pad0.98x0.95mm_HandSolder" (at 262.89 82.042 90)
-      (effects (font (size 1.27 1.27)) hide)
-    )
-    (property "Datasheet" "https://datasheet.lcsc.com/lcsc/1811151159_Resistor-Today-AECR0603F1K00K9_C328340.pdf" (at 262.89 83.82 0)
-      (effects (font (size 1.27 1.27)) hide)
-    )
-    (property "LCSC" "C328340" (at 262.89 83.82 90)
-      (effects (font (size 1.27 1.27)) hide)
-    )
-    (pin "1")
-    (pin "2")
-    (instances
-      (project "smoke_extractorV1_1"
-        (path "/9c1091b5-dc9c-4275-a62f-af3d6f92e0db"
-          (reference "R23") (unit 1)
-        )
-      )
-    )
-  )
   (symbol (lib_id "power:GND") (at 133.35 83.82 0) (unit 1)
     (in_bom yes) (on_board yes) (dnp no) (fields_autoplaced)
@@
     )
   )
+  (symbol (lib_id "Connector:Conn_01x01_Socket") (at 127 128.27 90) (unit 1)
+    (in_bom yes) (on_board yes) (dnp no)
+    (property "Reference" "J1" (at 125.73 126.365 90)
+      (effects (font (size 1.27 1.27)) (justify right))
+    )
+    (property "Value" "Conn_01x01_Socket" (at 120.65 127 0)
+      (effects (font (size 1.27 1.27)) (justify right))
+    )
+    (property "Footprint" "TestPoint:TestPoint_Pad_2.5x2.5mm" (at 127 128.27 0)
+      (effects (font (size 1.27 1.27)) hide)
+    )
+    (property "Datasheet" "~" (at 127 128.27 0)
+      (effects (font (size 1.27 1.27)) hide)
+    )
+    (pin "1")
+    (instances
+      (project "smoke_extractorV1_1"
+        (path "/9c1091b5-dc9c-4275-a62f-af3d6f92e0db"
+          (reference "J1") (unit 1)
+        )
+      )
+    )
+  )
   (symbol (lib_id "Mechanical:MountingHole_Pad") (at 127 167.64 0) (unit 1)
     (in_bom yes) (on_board yes) (dnp no) (fields_autoplaced)
@@
     )
   )
-  (symbol (lib_id "Connector:Conn_01x02_Socket") (at 127 128.27 90) (unit 1)
-    (in_bom yes) (on_board yes) (dnp no) (fields_autoplaced)
-    (property "Reference" "J13" (at 130.7592 128.905 90)
-      (effects (font (size 1.27 1.27)) (justify right))
-    )
-    (property "Value" "JST XH" (at 125.7808 127.6929 90)
-      (effects (font (face "KiCad Font") (size 1.27 1.27) bold (color 255 83 235 1)) (justify left) hide)
-    )
-    (property "Footprint" "Connector_JST:JST_PH_S2B-PH-K_1x02_P2.00mm_Horizontal" (at 127 128.27 0)
-      (effects (font (size 1.27 1.27)) hide)
-    )
-    (property "Datasheet" "https://www.lcsc.com/product-detail/Wire-To-Board-Wire-To-Wire-Connector_CAX-PH-2AW_C722769.html" (at 127 128.27 0)
-      (effects (font (size 1.27 1.27)) hide)
-    )
-    (property "LCSC" "C722769" (at 127 128.27 90)
-      (effects (font (size 1.27 1.27)) hide)
-    )
-    (pin "1")
-    (pin "2")
-    (instances
-      (project "bubblebutbot"
-        (path "/2cd1342d-9ef7-44f7-8a7d-ec49b5dc5750"
-          (reference "J13") (unit 1)
-        )
-      )
-      (project "smoke_extractorV1_1"
-        (path "/9c1091b5-dc9c-4275-a62f-af3d6f92e0db"
-          (reference "J1") (unit 1)
-        )
-      )
-    )
-  )
   (symbol (lib_id "Device:LED") (at 180.34 86.36 270) (unit 1)
     (in_bom yes) (on_board yes) (dnp no) (fields_autoplaced)
@@
   )
   (symbol (lib_id "power:PWR_FLAG") (at 127 134.62 90) (unit 1)
-    (in_bom yes) (on_board yes) (dnp no) (fields_autoplaced)
+    (in_bom yes) (on_board yes) (dnp no)
     (property "Reference" "#FLG0103" (at 125.095 134.62 0)
       (effects (font (size 1.27 1.27)) hide)
     )
-    (property "Value" "PWR_FLAG" (at 123.8251 135.0538 90)
-      (effects (font (size 1.27 1.27)) (justify left))
-    )
+    (property "Value" "PWR_FLAG" (at 123.19 137.16 0)
+      (effects (font (size 1.27 1.27)) (justify left))
+    )

Commit message: Version 2.05
Parts:
- removed C2: 120p, Capacitor_SMD:C_0603_1608Metric_Pad1.08x0.95mm_HandSolder, symbol Device:C
- removed C3, C4, C5: 10u, Capacitor_SMD:C_0603_1608Metric_Pad1.08x0.95mm_HandSolder, symbol Device:C
- removed D5: 3mmWhite, LED_THT:LED_D3.0mm, symbol Device:LED
- removed D6, D9: SS14, Diode_SMD:D_SMA, symbol Device:D_Schottky
- removed L2: 2.2u, Inductor_SMD:L_Coilcraft_LPS4018, symbol Device:L
- removed R17: 5, Resistor_SMD:R_0805_2012Metric_Pad1.20x1.40mm_HandSolder, symbol Device:R
- removed U4: TPS613222ADBV, Package_TO_SOT_SMD:SOT-23-5, symbol Regulator_Switching:TPS613222ADBV
- added D5: SS14, Diode_SMD:D_SMA, symbol Device:D_Schottky
- added D6: RLED, LED_SMD:LED_0603_1608Metric_Pad1.05x0.95mm_HandSolder, symbol Device:LED
- added F1: Fuse, Fuse:Fuse_0603_1608Metric_Pad1.05x0.95mm_HandSolder, symbol Device:Fuse
- D2, D3, D4: value 3mmWhite -> RLED; footprint LED_THT:LED_D3.0mm -> LED_SMD:LED_0603_1608Metric_Pad1.05x0.95mm_HandSolder; LCSC C86881 -> (none)
- SW1: footprint Button_Switch_SMD:SW_SPST_SKQG_WithStem -> Button_Switch_THT:SW_PUSH_6mm; LCSC C116647 -> (none)
Connections:
- net VBAT+PROTECT: now also U3.4 (VCC+), F1.2; no longer R20.1, U6.1 (V+)
- net VBUS: now also R1.1, TP2.1, D5.2 (A)
- net VSPLY: now also U2.1 (IN), D5.1 (K); no longer TP2.1
- net at R13.2: now also D3.2 (A); no longer D4.2 (A)
- net at D2.1 (K), D3.1 (K), D4.1 (K)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: now also D6.1 (K)
- net at R12.2: now also D4.2 (A)
- net at R14.2: now also D2.2 (A); no longer D3.2 (A)
- net at R15.2: now also D6.2 (A); no longer D2.2 (A)
- removed net +5V: R1.1, U2.1 (IN), U3.4 (VCC+)
- net V5_SWITCH renamed V_SWITCH
- new net: F1.1, R20.1, U6.1 (V+)
Other:
- note added: "A good candidate for a resetable fuse: https://www.lcsc.com/product-detail/Resettable-Fuses_BHFUSE-BSMD1206-100-16V_C883131.html"
- note added: "Max 1A!"
- note added: "While charging, the battery power is disabled"
- note removed: "Sch Diode 1A >"
- moved on the sheet: C1, D7, D8, Q1, R16, R18, R19, TP2, U5
