File: pcb/1v1/smoke_extractorV1_1.kicad_sch (KiCad schematic)
At the start: 50 parts, among them IC1 DW01A, J1 Conn_01x01_Socket, J2 Conn_01x01_Socket, Q1 FDN336P, SW1 SW_Push, U1 USB-TYPE-C-31-M-15, U2 SDDJE, U3 LM324DT, U5 TP4056, U6 18350-HOLDER, U7 ME2149FM5G, U8 FH8205

Commit message: v2.06
Parts:
- removed D6: RLED, LED_SMD:LED_0603_1608Metric_Pad1.05x0.95mm_HandSolder, symbol Device:LED
- removed R19: 1k, Resistor_SMD:R_0603_1608Metric_Pad0.98x0.95mm_HandSolder, symbol Device:R
- added C2: 0.1u, Capacitor_SMD:C_0603_1608Metric_Pad1.08x0.95mm_HandSolder, symbol Device:C
- added D9: RLED, LED_SMD:LED_0603_1608Metric_Pad1.05x0.95mm_HandSolder, symbol Device:LED
- added R7, R8: 3k3, Resistor_SMD:R_0603_1608Metric_Pad0.98x0.95mm_HandSolder, symbol Device:R
- D2: value RLED -> YLED
- D3, D4: value RLED -> GLED
- R1: value 3k6 -> 3k3; LCSC C103578 -> C3017726
- R11, R12, R14, R15, R18: value 1k -> 3k3; LCSC C328340 -> C3017726
- R13: value 1k -> 4k7; LCSC C328340 -> C105428
- R2: value 1k -> 5k1; LCSC C328340 -> C178023
Connections:
- net GND: now also R5.1, C2.2, D9.1 (K), R7.1; no longer R5.2, SW1.1
- net VBAT+PROTECT: now also SW1.2, C2.1; no longer U3.10 (POS_3), U3.12 (POS_4), U3.3 (POS_1), U3.4 (VCC+), U3.5 (POS_2)
- net VBUS: now also R18.1; no longer R1.1, R11.1
- net at D2.2 (A): now also D3.2 (A), D4.2 (A), R1.2, R13.1, SW1.1, U3.4 (VCC+); no longer R14.2
- net at U3.7 (OUT2): now also R12.2; no longer R13.1
- net at R13.2: now also U3.2 (NEG_1), U3.6 (NEG_2), U3.9 (NEG3), R7.2; no longer D3.2 (A)
- net at R11.2: now also U3.8 (OUT3); no longer D1.2 (A)
- net at D8.1 (K): now also R15.2
- net at U5.6 (~{STDBY}): now also R15.1
- net at D7.1 (K): now also R8.2; no longer R18.1
- net at U5.7 (~{CHRG}): now also R8.1; no longer R18.2
- net at U3.1 (OUT1): now also R14.2; no longer R12.1
- net at U3.14 (OUT4): no longer R15.1
- net at R14.1: now also D4.1 (K); no longer U3.8 (OUT3)
- new net: D2.1 (K), R11.1
- new net: D9.2 (A), R1.1, R2.1
- new net: D1.2 (A), R18.2
- new net: R4.1, R5.2, U3.10 (POS_3)
- new net: R2.2, R3.2, U3.3 (POS_1)
- new net: R3.1, R4.2, U3.5 (POS_2)
- new net: D3.1 (K), R12.1
- now unconnected: U3.13 (NEG_4)
- no-connect marks 6 -> 9
Other:
- note added: "1.32V @ 3.2V 1.73V @ 4.2V"
- note added: "1.34V (20)"
- note added: "1.48V (50)"
- note added: "1.64V (90)"
- note added: "2.3V drop"
- note removed: "3.9V"
- note removed: "3V"
- note removed: "Based on 5V"
- moved on the sheet: C1, D2, D3, D4, D5, D7, D8, Q1, R16, SW1, TP2, U3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
